Commit message: commit_message

File: src/mybot_description/urdf/mybot.xacro (robot description, xacro)
@@ -1,140 +1,246 @@
 <?xml version='1.0'?>
 <robot name="myrobot" xmlns:xacro="http://www.ros.org/wiki/xacro">
-  <xacro:property name="cameraSize" value="0.05"/>
-  <xacro:property name="cameraMass" value="0.1"/>
+  <xacro:property name="cameraSize" value="0.02"/>
+  <xacro:property name="cameraMass" value="0.001"/>
+  <xacro:property name="wheelMass" value="0.4"/>
   <xacro:include filename="$(find mybot_description)/urdf/mybot.gazebo" />
   <xacro:include filename="$(find mybot_description)/urdf/materials.xacro" />
-  <xacro:include filename="$(find mybot_description)/urdf/macros.xacro" />
-  <link name='chassis'>
-    <pose>0 0 0.1 0 0 0</pose>
-    <inertial>
-      <mass value="15.0"/>
-      <origin xyz="0.0 0 0.1" rpy=" 0 0 0"/>
-      <inertia
-          ixx="0.1" ixy="0" ixz="0"
-          iyy="0.1" iyz="0"
-          izz="0.1"
-      />
-    </inertial>
-    <collision name='collision'>
-      <geometry>
-        <box size=".4 .2 .1"/>
-      </geometry>
-    </collision>
-    <visual name='chassis_visual'>
-      <origin xyz="0 0 0" rpy=" 0 0 0"/>
-      <geometry>
-        <box size=".4 .2 .1"/>
-      </geometry>
-    </visual>
-    <collision name='caster_collision'>
-      <origin xyz="-0.15 0 -0.05" rpy=" 0 0 0"/>
-      <geometry>
-        <sphere radius="0.05"/>
-      </geometry>
-      <surface>
-        <friction>
-          <ode>
-            <mu>0</mu>
-            <mu2>0</mu2>
-            <slip1>1.0</slip1>
-            <slip2>1.0</slip2>
-          </ode>
-        </friction>
-      </surface>
-    </collision>
-    <visual name='caster_visual'>
-      <origin xyz="-0.15 0 -0.05" rpy=" 0 0 0"/>
-      <geometry>
-        <sphere radius="0.05"/>
-      </geometry>
-    </visual>
-    <collision name='caster_front_collision'>
-      <origin xyz="0.15 0 -0.05" rpy=" 0 0 0"/>
-      <geometry>
-        <sphere radius="0.05"/>
-      </geometry>
-      <surface>
-        <friction>
-          <ode>
-            <mu>0</mu>
-            <mu2>0</mu2>
-            <slip1>1.0</slip1>
-            <slip2>1.0</slip2>
-          </ode>
-        </friction>
-      </surface>
-    </collision>
-    <visual name='caster_front_visual'>
-      <origin xyz="0.15 0 -0.05" rpy=" 0 0 0"/>
-      <geometry>
-        <sphere radius="0.05"/>
-      </geometry>
-    </visual>
-  </link>
-  <link name="left_wheel">
-    <!--origin xyz="0.1 0.13 0.1" rpy="0 1.5707 1.5707"/-->
-    <collision name="collision">
-      <origin xyz="0 0 0" rpy="0 1.5707 1.5707"/>
-      <geometry>
-        <cylinder radius="0.1" length="0.05"/>
-      </geometry>
-    </collision>
-    <visual name="left_wheel_visual">
-      <origin xyz="0 0 0" rpy="0 1.5707 1.5707"/>
-      <geometry>
-        <cylinder radius="0.1" length="0.05"/>
-      </geometry>
-    </visual>
-    <inertial>
-      <origin xyz="0 0 0" rpy="0 1.5707 1.5707"/>
-      <mass value="5"/>
-      <inertia
-        ixx=".1" ixy="0.0" ixz="0.0"
-        iyy=".1" iyz="0.0"
-        izz=".1"/>
-    </inertial>
-  </link>
-  <link name="right_wheel">
-    <!--origin xyz="0.1 -0.13 0.1" rpy="0 1.5707 1.5707"/-->
-    <collision name="collision">
-      <origin xyz="0 0 0" rpy="0 1.5707 1.5707"/>
-      <geometry>
-        <cylinder radius="0.1" length="0.05"/>
-      </geometry>
-    </collision>
-    <visual name="right_wheel_visual">
-      <origin xyz="0 0 0" rpy="0 1.5707 1.5707"/>
-      <geometry>
-        <cylinder radius="0.1" length="0.05"/>
-      </geometry>
-    </visual>
-    <inertial>
-      <origin xyz="0 0 0" rpy="0 1.5707 1.5707"/>
-      <mass value="5"/>
-      <inertia
-        ixx=".1" ixy="0.0" ixz="0.0"
-        iyy=".1" iyz="0.0"
-        izz=".1"/>
-    </inertial>
-  </link>
-  <joint type="continuous" name="left_wheel_hinge">
-    <origin xyz="0 0.15 0" rpy="0 0 0"/>
-    <!--origin xyz="0.1 0.13 0" rpy="0 1.5707 1.5707"/-->
-    <child link="left_wheel"/>
-    <parent link="chassis"/>
-    <axis xyz="0 1 0" rpy="0 0 0"/>
-    <limit effort="10000" velocity="1000"/>
-    <joint_properties damping="1.0" friction="1.0"/>
-  </joint>
-  <joint type="continuous" name="right_wheel_hinge">
-    <origin xyz="0 -0.15 0" rpy="0 0 0"/>
-    <!--origin xyz="0.1 -0.13 0" rpy="0 1.5707 1.5707"/-->
-    <child link="right_wheel"/>
-    <parent link="chassis"/>
-    <axis xyz="0 1 0" rpy="0 0 0"/>
-    <limit effort="10000" velocity="1000"/>
-    <joint_properties damping="1.0" friction="1.0"/>
-  </joint>
+  <!--xacro:arg name="velodyne_points" default="true"/>
+  <xacro:arg name="front_laser_points" default="true"/>
+  <xacro:property name="front_laser_points" value="$(arg front_laser_points)"/>
+  <xacro:property name="velodyne_points" value="$(arg velodyne_points)"/>
+    <xacro:if value="${front_laser_points}">
+    	<xacro:include filename="$(find catvehicle)/urdf/catvehicle_front_laser_points.gazebo"/>
+    </xacro:if>
+    <xacro:if value="${velodyne_points}"-->
+      <!-- You can pass parameters in order to change the max/min
+           horizontal angles of the velodyne sensors. These are interpreted
+           in the velodyne_points gazebo file -->
+      <!--xacro:include filename="$(find catvehicle)/urdf/catvehicle_velodyne_points.gazebo"/>
+    </xacro:if>
+  <xacro:property name="sensor_box" value="0.25"/>
+  <xacro:property name="sensor_box2" value="0.31"/-->
+  <!--link name="base_footprint">
+    <inertial>
+      <mass value="0.0001"/>
+      <origin xyz="0 0 0"/>
+      <inertia ixx="0.0001" ixy="0.0" ixz="0.0" iyy="0.0001" iyz="0.0" izz="0.0001"/>
+    </inertial>
+    <visual>
+      <origin rpy="0 0 0" xyz="0 0 0"/>
+      <geometry>
+        <box size="0.001 0.001 0.001"/>
+      </geometry>
+    </visual>
+  </link>
+  <gazebo reference="base_footprint">
+    <turnGravityOff>false</turnGravityOff>
+  </gazebo>
+  <joint name="base_footprint_joint" type="fixed">
+    <origin rpy="0 0 0" xyz="0 0 0.04"/>
+    <parent link="base_footprint"/>
+    <child link="base_link"/>
+  </joint-->
+<link name="base_link">
+    <pose xyz="0 0 0.0" rpy="0 0 0" />
+  <inertial>
+    <mass value="10.0"/>
+    <origin xyz="0 0 0.05" rpy="0 0 0"/>
+    <inertia ixx="0.01632" ixy="0.0" ixz="0.0" iyy="0.01632" iyz="0.0" izz="0.01632"/>
+  </inertial>
+  <collision name='collision'>
+    <origin xyz="0 0 0.05" rpy="0 0 0" />
+    <geometry>
+      <box size="0.382 0.12 0.072"/>
+    </geometry>
+  </collision>
+  <visual name='base_link_visual'>
+    <origin xyz="0 0 0.05" rpy="0 0 0"/>
+    <geometry>
+      <!--box size="0.382 0.12 0.072"/-->
+      <box size="0.382 0.12 0.1"/>
+    </geometry>
+  </visual>
+</link>
+<joint type="continuous" name="joint_R1">
+  <parent link="base_link"/>
+  <child link="R1"/>
+  <origin xyz="0.1501 -0.0908 0" rpy="0 0 0"/>
+  <axis xyz="0 1 0" rpy="0 0 0"/>
+  <limit effort="10000" velocity="1000"/>
+  <joint_properties damping="1.0" friction="1.0"/>
+</joint>
+<link name="R1">
+  <collision name='collision'>
+    <origin xyz="0 0 0" rpy="0 1.5707 1.5707"/>
+    <geometry>
+      <cylinder radius="0.05" length="0.056"/>
+    </geometry>
+    <surface>
+      <friction>
+        <ode>
+          <mu>1</mu>
+          <mu2>1</mu2>
+          <slip1>0.5</slip1>
+          <slip2>0</slip2>
+        </ode>
+      </friction>
+    </surface>
+  </collision>
+  <visual name='R1_visual'>
+    <origin xyz="0 0 0" rpy="0 1.5707 1.5707"/>
+    <geometry>
+      <cylinder radius="0.05" length="0.056"/>
+    </geometry>
+  </visual>
+  <inertial>
+    <mass value="${wheelMass}"/>
+    <origin xyz="0 0 0" rpy="0 1.5707 1.5707"/>
+    <inertia ixx="0.035453" ixy="0.0" ixz="0.0" iyy="0.035453" iyz="0.0" izz="0.06272"/>
+  </inertial>
+</link>
+  <transmission name="R1_joint_trans">
+    <type>transmission_interface/SimpleTransmission</type>
+    <joint name="joint_R1"/>
+    <actuator name="R1_joint_motor">
+      <hardwareInterface>EffortJointInterface</hardwareInterface>
+      <mechanicalReduction>1</mechanicalReduction>
+    </actuator>
+  </transmission>
+<joint type="continuous" name="joint_R2">
+  <parent link="base_link"/>
+  <child link="R2"/>
+  <origin xyz="-0.1501 -0.0908 0" rpy="0 0 0"/>
+  <axis xyz="0 1 0" rpy="0 0 0"/>
+  <limit effort="10000" velocity="1000"/>
+  <joint_properties damping="1.0" friction="1.0"/>
+</joint>
+<link name="R2">
+  <collision name='collision'>
+    <origin xyz="0 0 0" rpy="0 1.5707 1.5707"/>
+    <geometry>
+      <cylinder radius="0.05" length="0.056"/>
+    </geometry>
+    <surface>
+      <friction>
+        <ode>
+          <mu>1</mu>
+          <mu2>1</mu2>
+          <slip1>0.5</slip1>
+          <slip2>0</slip2>
+        </ode>
+      </friction>
+    </surface>
+  </collision>
+  <visual name='R2_visual'>
+    <origin xyz="0 0 0" rpy="0 1.5707 1.5707"/>
+    <geometry>
+      <cylinder radius="0.05" length="0.056"/>
+    </geometry>
+  </visual>
+  <inertial>
+    <origin xyz="0 0 0" rpy="0 1.5707 1.5707"/>
+    <mass value="${wheelMass}"/>
+    <inertia ixx="0.035453" ixy="0.0" ixz="0.0" iyy="0.035453" iyz="0.0" izz="0.06272"/>
+  </inertial>
+</link>
+  <transmission name="R2_joint_trans">
+    <type>transmission_interface/SimpleTransmission</type>
+    <joint name="joint_R2"/>
+    <actuator name="R2_joint_motor">
+      <hardwareInterface>EffortJointInterface</hardwareInterface>
+      <mechanicalReduction>1</mechanicalReduction>
+    </actuator>
+  </transmission>
+<joint name="joint_L1" type="continuous">
+  <parent link="base_link"/>
+  <child link="L1"/>
+  <origin xyz="0.1501 0.0908 0" rpy="0 0 0"/>
+  <axis xyz="0 1 0"/>
+  <limit effort="10000" velocity="1000"/>
+  <joint_properties damping="1.0" friction="1.0"/>
+</joint>
+<link name="L1">
+  <collision name='collision'>
+    <origin xyz="0 0 0" rpy="0 1.5707 1.5707"/>
+    <geometry>
+      <cylinder radius="0.05" length="0.056"/>
+    </geometry>
+    <surface>
+      <friction>
+        <ode>
+          <mu>1</mu>
+          <mu2>1</mu2>
+          <slip1>0.5</slip1>
+          <slip2>0</slip2>
+        </ode>
+      </friction>
+    </surface>
+  </collision>
+  <visual name='L1_visual'>
+    <origin xyz="0 0 0" rpy="0 1.5707 1.5707"/>
+    <geometry>
+      <cylinder radius="0.05" length="0.056"/>
+    </geometry>
+  </visual>
+  <inertial>
+    <origin xyz="0 0 0" rpy="0 1.5707 1.5707"/>
+    <mass value="${wheelMass}"/>
+    <inertia ixx="0.035453" ixy="0.0" ixz="0.0" iyy="0.035453" iyz="0.0" izz="0.06272"/>
+    </inertial>
+</link>
+  <transmission name="L1_joint_trans">
+    <type>transmission_interface/SimpleTransmission</type>
+    <joint name="joint_L1"/>
+    <actuator name="L1_joint_motor">
+      <hardwareInterface>EffortJointInterface</hardwareInterface>
+      <mechanicalReduction>1</mechanicalReduction>
+    </actuator>
+  </transmission>
+<joint name="joint_L2" type="continuous">
+  <parent link="base_link"/>
+  <child link="L2"/>
+  <origin xyz="-0.1501 0.0908 0" rpy="0 0 0" />
+  <axis xyz="0 1 0" rpy="0 0 0"/>
+  <limit effort="10000" velocity="1000"/>
+  <joint_properties damping="1.0" fiction="1.0"/>
+</joint>
+<link name="L2">
+  <collision name='collision'>
+    <origin xyz="0 0 0" rpy="0 1.5707 1.5707"/>
+    <geometry>
+      <cylinder radius="0.05" length="0.056"/>
+    </geometry>
+    <surface>
+      <friction>
+        <ode>
+          <mu>1</mu>
+          <mu2>1</mu2>
+          <slip1>0.5</slip1>
+          <slip2>0</slip2>
+        </ode>
+      </friction>
+    </surface>
+  </collision>
+  <visual name='L2_visual'>
+    <origin xyz="0 0 0" rpy="0 1.5707 1.5707"/>
+    <geometry>
+      <cylinder radius="0.05" length="0.056"/>
+    </geometry>
+  </visual>
+  <inertial>
+    <origin xyz="0 0 0" rpy="0 1.5707 1.5707"/>
+    <mass value="${wheelMass}"/>
+    <inertia ixx="0.035453" ixy="0.0" ixz="0.0" iyy="0.035453" iyz="0.0" izz="0.06272"/>
+  </inertial>
+</link>
+  <transmission name="L2_joint_trans">
+    <type>transmission_interface/SimpleTransmission</type>
+    <joint name="joint_L2"/>
+    <actuator name="L2_joint_motor">
+      <hardwareInterface>EffortJointInterface</hardwareInterface>
+      <mechanicalReduction>1</mechanicalReduction>
+    </actuator>
+  </transmission>
   <link name="camera">
     <collision>
@@ -160,12 +266,149 @@
   <joint name="camera_joint" type="fixed">
     <axis xyz="0 1 0" />
-    <origin xyz=".2 0 0" rpy="0 0 0"/>
-    <parent link="chassis"/>
+    <!--origin xyz="0.2015 0 0.05" rpy="0 0 0"/-->
+    <origin xyz="0.2015 0 0.085" rpy="0 0 0"/>
+    <parent link="base_link"/>
     <child link="camera"/>
   </joint>
+  <!--link name="camera2">
+    <collision>
+      <origin xyz="0 0 0" rpy="0 0 0"/>
+      <geometry>
+        <box size="${cameraSize} ${cameraSize} ${cameraSize}"/>
+      </geometry>
+    </collision>
+    <visual>
+      <origin xyz="0 0 0" rpy="0 0 0"/>
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
Commit message: commmmit

File: src/mybot_description/urdf/mybot.xacro (robot description, xacro)
@@ -52,5 +52,6 @@
     <origin xyz="0 0 0.05" rpy="0 0 0" />
     <geometry>
-      <box size="0.382 0.12 0.072"/>
+      <!--box size="0.382 0.12 0.072"/-->
+      <box size="0.382 0.12 0.1"/>
     </geometry>
   </collision>
@@ -409,5 +410,5 @@
   <joint name="hokuyo_joint" type="fixed">
     <axis xyz="0 1 0" />
-    <origin xyz="0.2215 0 0.035" rpy="0 0 0"/>
+    <origin xyz="0.0 0 0.122" rpy="0 0 0"/>
     <parent link="base_link"/>
     <child link="hokuyo"/>
@@ -416,5 +417,5 @@
   <link name="hokuyo">
     <collision>
-      <origin xyz="0 0 0" rpy="0 1.5707 0"/>
+      <origin xyz="0 0 0" rpy="0 0 0"/>
       <geometry>
     <box size="0.1 0.1 0.1"/>
@@ -422,5 +423,5 @@
     </collision>
     <visual>
-      <origin xyz="0 0 0" rpy="0 1.5707 0"/>
+      <origin xyz="0 0 0" rpy="0 0 0"/>
       <geometry>
         <mesh filename="package://mybot_description/meshes/hokuyo.dae"/>
@@ -473,5 +474,5 @@
         <sphere radius="0.025"/>
       </geometry>
-      <origin rpy="1.57079632679 0 0" xyz="0 0.02 0 "/>
+      <origin rpy="1.57079632679 0 0" xyz="0.02 0.02 0 "/>
     </collision>
     <inertial>

Commit message: myworld

File: src/mybot_description/urdf/mybot.xacro (robot description, xacro)
@@ -3,5 +3,5 @@
   <xacro:property name="cameraSize" value="0.02"/>
   <xacro:property name="cameraMass" value="0.001"/>
-  <xacro:property name="wheelMass" value="0.4"/>
+  <xacro:property name="wheelMass" value="1.0"/>
   <xacro:include filename="$(find mybot_description)/urdf/mybot.gazebo" />
   <xacro:include filename="$(find mybot_description)/urdf/materials.xacro" />
@@ -43,12 +43,12 @@
   </joint-->
 <link name="base_link">
-    <pose xyz="0 0 0.0" rpy="0 0 0" />
+    <pose xyz="0 0 0" rpy="0 0 0" />
   <inertial>
     <mass value="10.0"/>
-    <origin xyz="0 0 0.05" rpy="0 0 0"/>
+    <origin xyz="0 0 0.3" rpy="0 0 0"/>
     <inertia ixx="0.01632" ixy="0.0" ixz="0.0" iyy="0.01632" iyz="0.0" izz="0.01632"/>
   </inertial>
   <collision name='collision'>
-    <origin xyz="0 0 0.05" rpy="0 0 0" />
+    <origin xyz="0 0 0.3" rpy="0 0 0" />
     <geometry>
       <!--box size="0.382 0.12 0.072"/-->
@@ -57,5 +57,5 @@
   </collision>
   <visual name='base_link_visual'>
-    <origin xyz="0 0 0.05" rpy="0 0 0"/>
+    <origin xyz="0 0 0.3" rpy="0 0 0"/>
     <geometry>
       <!--box size="0.382 0.12 0.072"/-->
@@ -67,5 +67,5 @@
   <parent link="base_link"/>
   <child link="R1"/>
-  <origin xyz="0.1501 -0.0908 0" rpy="0 0 0"/>
+  <origin xyz="0.1501 -0.0908 0.25" rpy="0 0 0"/>
   <axis xyz="0 1 0" rpy="0 0 0"/>
   <limit effort="10000" velocity="1000"/>
@@ -74,5 +74,5 @@
 <link name="R1">
   <collision name='collision'>
-    <origin xyz="0 0 0" rpy="0 1.5707 1.5707"/>
+    <origin xyz="0 0 0" rpy="0 1.57079632679 1.57079632679"/>
     <geometry>
       <cylinder radius="0.05" length="0.056"/>
@@ -90,5 +90,5 @@
   </collision>
   <visual name='R1_visual'>
-    <origin xyz="0 0 0" rpy="0 1.5707 1.5707"/>
+    <origin xyz="0 0 0" rpy="0 1.57079632679 1.57079632679"/>
     <geometry>
       <cylinder radius="0.05" length="0.056"/>
@@ -97,5 +97,5 @@
   <inertial>
     <mass value="${wheelMass}"/>
-    <origin xyz="0 0 0" rpy="0 1.5707 1.5707"/>
+    <origin xyz="0 0 0" rpy="0 1.57079632679 1.57079632679"/>
     <inertia ixx="0.035453" ixy="0.0" ixz="0.0" iyy="0.035453" iyz="0.0" izz="0.06272"/>
   </inertial>
@@ -112,5 +112,5 @@
   <parent link="base_link"/>
   <child link="R2"/>
-  <origin xyz="-0.1501 -0.0908 0" rpy="0 0 0"/>
+  <origin xyz="-0.1501 -0.0908 0.25" rpy="0 0 0"/>
   <axis xyz="0 1 0" rpy="0 0 0"/>
   <limit effort="10000" velocity="1000"/>
@@ -119,5 +119,5 @@
 <link name="R2">
   <collision name='collision'>
-    <origin xyz="0 0 0" rpy="0 1.5707 1.5707"/>
+    <origin xyz="0 0 0" rpy="0 1.57079632679 1.57079632679"/>
     <geometry>
       <cylinder radius="0.05" length="0.056"/>
@@ -135,5 +135,5 @@
   </collision>
   <visual name='R2_visual'>
-    <origin xyz="0 0 0" rpy="0 1.5707 1.5707"/>
+    <origin xyz="0 0 0" rpy="0 1.57079632679 1.57079632679"/>
     <geometry>
       <cylinder radius="0.05" length="0.056"/>
@@ -141,5 +141,5 @@
   </visual>
   <inertial>
-    <origin xyz="0 0 0" rpy="0 1.5707 1.5707"/>
+    <origin xyz="0 0 0" rpy="0 1.57079632679 1.57079632679"/>
     <mass value="${wheelMass}"/>
     <inertia ixx="0.035453" ixy="0.0" ixz="0.0" iyy="0.035453" iyz="0.0" izz="0.06272"/>
@@ -157,5 +157,5 @@
   <parent link="base_link"/>
   <child link="L1"/>
-  <origin xyz="0.1501 0.0908 0" rpy="0 0 0"/>
+  <origin xyz="0.1501 0.0908 0.25" rpy="0 0 0"/>
   <axis xyz="0 1 0"/>
   <limit effort="10000" velocity="1000"/>
@@ -164,5 +164,5 @@
 <link name="L1">
   <collision name='collision'>
-    <origin xyz="0 0 0" rpy="0 1.5707 1.5707"/>
+    <origin xyz="0 0 0" rpy="0 1.57079632679 1.57079632679"/>
     <geometry>
       <cylinder radius="0.05" length="0.056"/>
@@ -180,5 +180,5 @@
   </collision>
   <visual name='L1_visual'>
-    <origin xyz="0 0 0" rpy="0 1.5707 1.5707"/>
+    <origin xyz="0 0 0" rpy="0 1.57079632679 1.57079632679"/>
     <geometry>
       <cylinder radius="0.05" length="0.056"/>
@@ -186,5 +186,5 @@
   </visual>
   <inertial>
-    <origin xyz="0 0 0" rpy="0 1.5707 1.5707"/>
+    <origin xyz="0 0 0" rpy="0 1.57079632679 1.57079632679"/>
     <mass value="${wheelMass}"/>
     <inertia ixx="0.035453" ixy="0.0" ixz="0.0" iyy="0.035453" iyz="0.0" izz="0.06272"/>
@@ -202,5 +202,5 @@
   <parent link="base_link"/>
   <child link="L2"/>
-  <origin xyz="-0.1501 0.0908 0" rpy="0 0 0" />
+  <origin xyz="-0.1501 0.0908 0.25" rpy="0 0 0" />
   <axis xyz="0 1 0" rpy="0 0 0"/>
   <limit effort="10000" velocity="1000"/>
@@ -209,5 +209,5 @@
 <link name="L2">
   <collision name='collision'>
-    <origin xyz="0 0 0" rpy="0 1.5707 1.5707"/>
+    <origin xyz="0 0 0" rpy="0 1.57079632679 1.57079632679"/>
     <geometry>
       <cylinder radius="0.05" length="0.056"/>
@@ -225,5 +225,5 @@
   </collision>
   <visual name='L2_visual'>
-    <origin xyz="0 0 0" rpy="0 1.5707 1.5707"/>
+    <origin xyz="0 0 0" rpy="0 1.57079632679 1.57079632679"/>
     <geometry>
       <cylinder radius="0.05" length="0.056"/>
@@ -231,5 +231,5 @@
   </visual>
   <inertial>
-    <origin xyz="0 0 0" rpy="0 1.5707 1.5707"/>
+    <origin xyz="0 0 0" rpy="0 1.57079632679 1.57079632679"/>
     <mass value="${wheelMass}"/>
     <inertia ixx="0.035453" ixy="0.0" ixz="0.0" iyy="0.035453" iyz="0.0" izz="0.06272"/>
@@ -268,5 +268,5 @@
     <axis xyz="0 1 0" />
     <!--origin xyz="0.2015 0 0.05" rpy="0 0 0"/-->
-    <origin xyz="0.2015 0 0.085" rpy="0 0 0"/>
+    <origin xyz="0.2015 0 0.3" rpy="0 0 0"/>
     <parent link="base_link"/>
     <child link="camera"/>
@@ -410,5 +410,5 @@
   <joint name="hokuyo_joint" type="fixed">
     <axis xyz="0 1 0" />
-    <origin xyz="0.0 0 0.122" rpy="0 0 0"/>
+    <origin xyz="0.0 0 0.372" rpy="0 0 0"/>
     <parent link="base_link"/>
     <child link="hokuyo"/>
@@ -457,5 +457,5 @@
     <parent link="base_link"/>
     <child link="caster_front_link"/>
-    <origin rpy="-1.57079632679 0 0" xyz="0.115 0.0 0.007"/>
+    <origin rpy="-1.57079632679 0 0" xyz="0.115 0.0 0.257"/>
   </joint>
   <gazebo reference="caster_front_link">
@@ -485,5 +485,5 @@
     <parent link="base_link"/>
     <child link="caster_back_link"/>
-    <origin rpy="-1.57079632679 0 0" xyz="-0.135 0.0 0.009"/>
+    <origin rpy="-1.57079632679 0 0" xyz="-0.135 0.0 0.257"/>
   </joint>
   <gazebo reference="caster_back_link">

File: src/mybot_gazebo/worlds/파트1.SLDPRT.urdf (robot description, URDF)
Before this commit: robot 파트1.SLDPRT, 1 links, 0 joints
Links:
- removed link part.SLDPRT
- added link 파트1.SLDPRT, mass 1733100; collision mesh filename=package://파트1.SLDPRT/meshes/파트1.SLDPRT.STL; visual mesh filename=package://파트1.SLDPRT/meshes/파트1.SLDPRT.STL
