Commit message: commit

File: src/mybot_description/urdf/mybot.xacro (robot description, xacro)
@@ -6,40 +6,4 @@
   <xacro:include filename="$(find mybot_description)/urdf/mybot.gazebo" />
   <xacro:include filename="$(find mybot_description)/urdf/materials.xacro" />
-  <!--xacro:arg name="velodyne_points" default="true"/>
-  <xacro:arg name="front_laser_points" default="true"/>
-  <xacro:property name="front_laser_points" value="$(arg front_laser_points)"/>
-  <xacro:property name="velodyne_points" value="$(arg velodyne_points)"/>
-    <xacro:if value="${front_laser_points}">
-    	<xacro:include filename="$(find catvehicle)/urdf/catvehicle_front_laser_points.gazebo"/>
-    </xacro:if>
-    <xacro:if value="${velodyne_points}"-->
-      <!-- You can pass parameters in order to change the max/min
-           horizontal angles of the velodyne sensors. These are interpreted
-           in the velodyne_points gazebo file -->
-      <!--xacro:include filename="$(find catvehicle)/urdf/catvehicle_velodyne_points.gazebo"/>
-    </xacro:if>
-  <xacro:property name="sensor_box" value="0.25"/>
-  <xacro:property name="sensor_box2" value="0.31"/-->
-  <!--link name="base_footprint">
-    <inertial>
-      <mass value="0.0001"/>
-      <origin xyz="0 0 0"/>
-      <inertia ixx="0.0001" ixy="0.0" ixz="0.0" iyy="0.0001" iyz="0.0" izz="0.0001"/>
-    </inertial>
-    <visual>
-      <origin rpy="0 0 0" xyz="0 0 0"/>
-      <geometry>
-        <box size="0.001 0.001 0.001"/>
-      </geometry>
-    </visual>
-  </link>
-  <gazebo reference="base_footprint">
-    <turnGravityOff>false</turnGravityOff>
-  </gazebo>
-  <joint name="base_footprint_joint" type="fixed">
-    <origin rpy="0 0 0" xyz="0 0 0.04"/>
-    <parent link="base_footprint"/>
-    <child link="base_link"/>
-  </joint-->
 <link name="base_link">
     <pose xyz="0 0 0" rpy="0 0 0" />
@@ -52,5 +16,4 @@
     <origin xyz="0 0 0.3" rpy="0 0 0" />
     <geometry>
-      <!--box size="0.382 0.12 0.072"/-->
       <box size="0.382 0.12 0.1"/>
     </geometry>
@@ -59,5 +22,4 @@
     <origin xyz="0 0 0.3" rpy="0 0 0"/>
     <geometry>
-      <!--box size="0.382 0.12 0.072"/-->
       <box size="0.382 0.12 0.1"/>
     </geometry>
@@ -267,145 +229,9 @@
   <joint name="camera_joint" type="fixed">
     <axis xyz="0 1 0" />
-    <!--origin xyz="0.2015 0 0.05" rpy="0 0 0"/-->
     <origin xyz="0.2015 0 0.3" rpy="0 0 0"/>
     <parent link="base_link"/>
     <child link="camera"/>
   </joint>
-  <!--link name="camera2">
-    <collision>
-      <origin xyz="0 0 0" rpy="0 0 0"/>
-      <geometry>
-        <box size="${cameraSize} ${cameraSize} ${cameraSize}"/>
-      </geometry>
-    </collision>
-    <visual>
-      <origin xyz="0 0 0" rpy="0 0 0"/>
-      <geometry>
-        <box size="${cameraSize} ${cameraSize} ${cameraSize}"/>
-      </geometry>
-      <material name="green"/>
-    </visual>
-    <inertial>
-      <mass value="${cameraMass}" />
-      <origin xyz="0 0 0" rpy="0 0 0"/>
-      <box_inertia m="0.000000001" x="${cameraSize}" y="${cameraSize}" z="${cameraSize}" />
-      <inertia ixx="1e-6" ixy="0" ixz="0" iyy="1e-6" iyz="0" izz="1e-6" />
-    </inertial>
-  </link>
-  <joint name="camera2_joint" type="fixed">
-    <axis xyz="0 1 0" />
-    <origin xyz="0.2015 0.03 0.05" rpy="0 0 0"/>
-    <parent link="base_link"/>
-    <child link="camera2"/>
-  </joint-->
-<!--joint name="cameraLeft_joint" type="fixed">
-    <origin xyz=".2015 -0.05 0.05" rpy="0 0 0"/>
-    <parent link="base_link"/>
-    <child link="cameraLeft_link"/>
-  </joint>
-  <link name="cameraLeft_link">
-    <collision>
-      <origin xyz="0 0 0" rpy="0 0 0"/>
-      <geometry>
-        <box size="0.02 0.02 0.02"/>
-      </geometry>
-    </collision>
-    <visual>
-      <origin xyz="0 0 0" rpy="0 0 0"/>
-      <geometry>
-    <box size="0.02 0.02 0.02"/>
-      </geometry>
-      <material name="orange"/>
-    </visual>
-    <inertial>
-      <origin xyz="0 0 0" rpy="0 0 0"/>
-      <mass value="0.001"/>
-      <box_inertia m="0.001" x="0.02" y="0.02" z="0.02"/>
-      <inertia ixx="1e-6" ixy="0" ixz="0" iyy="1e-6" iyz="0" izz="1e-6" />
-    </inertial>
-  </link>
-  <joint name="cameraLeft_depth_joint" type="fixed">
-    <origin xyz="0 0 0" rpy="-1.5707 0 -1.5707 "/>
-    <parent link="cameraLeft_link"/>
-    <child link="cameraLeft_depth_link"/>
-  </joint>
-  <link name="cameraLeft_depth_link"></link-->
-<!--joint name="camera_joint" type="fixed">
-<origin xyz="0 0 0.121" rpy="0 0 0"/>
-	<axis xyz="0 0 1"/>
-	<parent link="base_link"/>
-	<child link="camera_link"/>
-</joint>
-<link name="camera_link">
-	<collision>
-	  <origin xyz="0 0 0" rpy="0 0 0"/>
-	  <geometry>
-	   <box size="${sensor_box} ${sensor_box} ${sensor_box}"/>
-	  </geometry>
-	</collision>
-	<visual>
-	  <origin xyz="0 0 0" rpy="0 0 0"/>
-	  <geometry>
-	  <box size="${sensor_box} ${sensor_box} ${sensor_box}"
-/>
-          </geometry>
-	</visual>
-    <inertial>
-      <mass value="1e-5" />
-      <origin xyz="0 0 0" rpy="0 0 0"/>
-      <inertia ixx="1e-6" ixy="0" ixz="0" iyy="1e-6" iyz="0" izz="1e-6" />
-    </inertial>
-</link>
-<joint name="velodyne_joint" type="fixed">
-	<origin xyz="0 0 1.965" rpy="0 0 0"/>
-	<axis xyz="0 0 1"/>
-	<parent link="camera_link"/>
-	<child link="velodyne_link"/>
-</joint>
-<link name="velodyne_link">
-        <collision>
-          <origin xyz="0 0 0" rpy="0 0 0"/>
-          <geometry>
-           <box size="0.1 0.1 0.1"/>
-          </geometry>
-        </collision>
-        <visual>
-          <origin xyz="0 0 0" rpy="0 0 0"/>
-          <geometry>
-           <box size="${sensor_box} ${sensor_box} ${sensor_box}"/>
-          </geometry>
-        </visual>
-    <inertial>
-      <mass value="1e-5" />
-      <origin xyz="0 0 0" rpy="0 0 0"/>
-      <inertia ixx="1e-6" ixy="0" ixz="0" iyy="1e-6" iyz="0" izz="1e-6" />
-    </inertial>
-</link>
-<joint name="front_laser_joint" type="fixed">
-	<origin xyz="0 0 2" rpy="0 0 0"/>
-	<axis xyz="0 0 1"/>
-	<parent link="base_link"/>
-	<child link="front_laser_link"/>
-</joint>
-<link name="front_laser_link">
-     <parent link="front_laser_joint"/>
-        <collision>
-          <origin xyz="0 0 0" rpy="0 0.0 0"/>
-          <geometry>
-           <box size="${sensor_box} ${sensor_box} ${sensor_box}"/>
-          </geometry>
-        </collision>
-        <visual>
-          <origin xyz="0 0 0" rpy="0 0 0"/>
-          <geometry>
-           <box size="${sensor_box} ${sensor_box} ${sensor_box}"/>
-          </geometry>
-        </visual>
-    <inertial>
-      <mass value="1e-5" />
-      <origin xyz="0 0 0" rpy="0 0 0"/>
-      <inertia ixx="1e-6" ixy="0" ixz="0" iyy="1e-6" iyz="0" izz="1e-6" />
-    </inertial>
-</link-->
+  <!-- Hokuyo Laser -->
   <joint name="hokuyo_joint" type="fixed">
     <axis xyz="0 1 0" />
@@ -414,5 +240,4 @@
     <child link="hokuyo"/>
   </joint>
-  <!-- Hokuyo Laser -->
   <link name="hokuyo">
     <collision>
